File: layouts/default/default.kicad_pcb (KiCad board)
At the start: 2 copper layers, 22 parts

Commit message: V1, added pubishing info
Parts:
- moved LED2 386.0 mm to (191.5, 125.1), turned to 90 degrees
- moved C8 375.2 mm to (195.2, 120.4)
- moved C3 360.1 mm to (189.9, 116.0), turned to 180 degrees
- moved C4 347.5 mm to (187.9, 112.3), turned to -90 degrees
- moved R3 344.3 mm to (189.9, 117.2), turned to 180 degrees
- moved R8 339.3 mm to (192.3, 119.5)
- moved R1 323.8 mm to (190.3, 111.9), turned to -90 degrees
- moved R9 318.5 mm to (197.2, 120.1), turned to 90 degrees
- moved C5 315.5 mm to (193.7, 109.0), turned to 180 degrees
- moved R5 299.1 mm to (193.7, 108.0), turned to 180 degrees
- moved R4 294.0 mm to (189.6, 114.8)
- moved LED4 293.8 mm to (200.2, 125.0), turned to 90 degrees
- moved C1 290.8 mm to (192.4, 118.1), turned to 180 degrees
- moved LED3 283.6 mm to (195.8, 125.1), turned to 90 degrees
- moved LED1 270.4 mm to (187.2, 125.1), turned to 90 degrees
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Connections:
- C2 pad 1: C3-net -> VCC
- C2 pad 2: C3-net-1 -> gnd
- C3 pad 2: net -> net-1
- C7 pad 1: unnamed[0] -> net
- C8 pad 1: unnamed[0] -> net
- R4 pad 1: net -> net-1
- R8 pad 2: unnamed[0] -> net
Routing:
- net gnd: track 0.00 -> 50.6 mm, vias 0 -> 3
- net K: track 0.00 -> 23.1 mm
- net OUT2: track 0.00 -> 13.2 mm, vias 0 -> 2
- net IN2minus: track 0.00 -> 11.3 mm, vias 0 -> 2
- net IN2plus: track 0.00 -> 10.4 mm
- net IN1plus: track 0.00 -> 7.96 mm
- net VCC: track 0.00 -> 6.56 mm
- net OUT1: track 0.00 -> 5.03 mm
- net net: track 0.00 -> 2.82 mm
- net out: track 0.00 -> 1.42 mm
- net net-1: track 0.00 -> 1.23 mm
